File: LedClock.sch (KiCad schematic (older format))
At the start: 148 parts, among them J1 USB_B_Micro, J2 STM32_Debug, Q1 NJL7502R, SW1 Rotary_Encoder, U1 PCA9635, U2 PCA9635, U3 PCA9635, U4 PCA9635, U5 NJM78L33SU3, U6 STM32F303K8Tx, X1 12MHz

Commit message: 基板 V1.1
Parts:
- removed J2: STM32_Debug, Connector_PinHeader_1.27mm:PinHeader_2x05_P1.27mm_Vertical, symbol LedClock:STM32_Debug
- added J2: STM32_Debug, LedClock:STM32_Debug_5pin, symbol LedClock:STM32_Debug_5pin
Connections:
- net +3V3: now also J2.3 (VDD)
- net +5V: now also D1.2 (A), D10.2 (A), D11.2 (A), D12.2 (A), D13.2 (A), D14.2 (A), D15.2 (A), D16.2 (A), D17.2 (A), D18.2 (A), D19.2 (A), D2.2 (A), D20.2 (A), D21.2 (A), D22.2 (A), D23.2 (A), D24.2 (A), D25.2 (A), D26.2 (A), D27.2 (A), D28.2 (A), D29.2 (A), D3.2 (A), D30.2 (A), D31.2 (A), D32.2 (A), D33.2 (A), D34.2 (A), D35.2 (A), D36.2 (A), D37.2 (A), D38.2 (A), D39.2 (A), D4.2 (A), D40.2 (A), D41.2 (A), D42.2 (A), D43.2 (A), D44.2 (A), D45.2 (A), D46.2 (A), D47.2 (A), D48.2 (A), D49.2 (A), D5.2 (A), D50.2 (A), D51.2 (A), D52.2 (A), D53.2 (A), D54.2 (A), D55.2 (A), D56.2 (A), D57.2 (A), D58.2 (A), D59.2 (A), D6.2 (A), D60.2 (A), D7.2 (A), D8.2 (A), D9.2 (A); no longer R1.1, R10.1, R11.1, R12.1, R13.1, R14.1, R15.1, R16.1, R17.1, R18.1, R19.1, R2.1, R20.1, R21.1, R22.1, R23.1, R24.1, R25.1, R26.1, R27.1, R28.1, R29.1, R3.1, R30.1, R31.1, R32.1, R33.1, R34.1, R35.1, R36.1, R37.1, R38.1, R39.1, R4.1, R40.1, R41.1, R42.1, R43.1, R44.1, R45.1, R46.1, R47.1, R48.1, R49.1, R5.1, R50.1, R51.1, R52.1, R53.1, R54.1, R55.1, R56.1, R57.1, R58.1, R59.1, R6.1, R60.1, R7.1, R8.1, R9.1
- net GND: now also J2.1 (GND)
- net NRST: now also J2.2 (NRST)
- net SWDIO: now also J2.5 (SWDIO)
- net at U1.10 (LED4): now also R5.2; no longer D5.1 (K)
- net at U1.11 (LED5): now also R6.2; no longer D6.1 (K)
- net at U1.12 (LED6): now also R7.2; no longer D7.1 (K)
- net at U1.13 (LED7): now also R8.2; no longer D8.1 (K)
- net at U1.15 (LED8): now also R9.2; no longer D9.1 (K)
- net at U1.16 (LED9): now also R10.2; no longer D10.1 (K)
- net at U1.17 (LED10): now also R11.2; no longer D11.1 (K)
- net at U1.18 (LED11): now also R12.2; no longer D12.1 (K)
- net at U1.19 (LED12): now also R13.2; no longer D13.1 (K)
- net at U1.20 (LED13): now also R14.2; no longer D14.1 (K)
- net at U1.21 (LED14): now also R15.2; no longer D15.1 (K)
- net at U1.6 (LED0): now also R1.2; no longer D1.1 (K)
- net at U1.7 (LED1): now also R2.2; no longer D2.1 (K)
- net at U1.8 (LED2): now also R3.2; no longer D3.1 (K)
- net at U1.9 (LED3): now also R4.2; no longer D4.1 (K)
- net at U2.10 (LED4): now also R20.2; no longer D20.1 (K)
- net at U2.11 (LED5): now also R21.2; no longer D21.1 (K)
- net at U2.12 (LED6): now also R22.2; no longer D22.1 (K)
- net at U2.13 (LED7): now also R23.2; no longer D23.1 (K)
- net at U2.15 (LED8): now also R24.2; no longer D24.1 (K)
- net at U2.16 (LED9): now also R25.2; no longer D25.1 (K)
- net at U2.17 (LED10): now also R26.2; no longer D26.1 (K)
- net at U2.18 (LED11): now also R27.2; no longer D27.1 (K)
- net at U2.19 (LED12): now also R28.2; no longer D28.1 (K)
- net at U2.20 (LED13): now also R29.2; no longer D29.1 (K)
- net at U2.21 (LED14): now also R30.2; no longer D30.1 (K)
- net at U2.6 (LED0): now also R16.2; no longer D16.1 (K)
- net at U2.7 (LED1): now also R17.2; no longer D17.1 (K)
- net at U2.8 (LED2): now also R18.2; no longer D18.1 (K)
- net at U2.9 (LED3): now also R19.2; no longer D19.1 (K)
- net at U3.10 (LED4): now also R35.2; no longer D35.1 (K)
- net at U3.11 (LED5): now also R36.2; no longer D36.1 (K)
- net at U3.12 (LED6): now also R37.2; no longer D37.1 (K)
- net at U3.13 (LED7): now also R38.2; no longer D38.1 (K)
- net at U3.15 (LED8): now also R39.2; no longer D39.1 (K)
- net at U3.16 (LED9): now also R40.2; no longer D40.1 (K)
- net at U3.17 (LED10): now also R41.2; no longer D41.1 (K)
- net at U3.18 (LED11): now also R42.2; no longer D42.1 (K)
- net at U3.19 (LED12): now also R43.2; no longer D43.1 (K)
- net at U3.20 (LED13): now also R44.2; no longer D44.1 (K)
- net at U3.21 (LED14): now also R45.2; no longer D45.1 (K)
- net at U3.6 (LED0): now also R31.2; no longer D31.1 (K)
- net at U3.7 (LED1): now also R32.2; no longer D32.1 (K)
- net at U3.8 (LED2): now also R33.2; no longer D33.1 (K)
- net at U3.9 (LED3): now also R34.2; no longer D34.1 (K)
- net at U4.10 (LED4): now also R50.2; no longer D50.1 (K)
- net at U4.11 (LED5): now also R51.2; no longer D51.1 (K)
- net at U4.12 (LED6): now also R52.2; no longer D52.1 (K)
- net at U4.13 (LED7): now also R53.2; no longer D53.1 (K)
- net at U4.15 (LED8): now also R54.2; no longer D54.1 (K)
- net at U4.16 (LED9): now also R55.2; no longer D55.1 (K)
- net at U4.17 (LED10): now also R56.2; no longer D56.1 (K)
- net at U4.18 (LED11): now also R57.2; no longer D57.1 (K)
- net at U4.19 (LED12): now also R58.2; no longer D58.1 (K)
- net at U4.20 (LED13): now also R59.2; no longer D59.1 (K)
- net at U4.21 (LED14): now also R60.2; no longer D60.1 (K)
- net at U4.6 (LED0): now also R46.2; no longer D46.1 (K)
- net at U4.7 (LED1): now also R47.2; no longer D47.1 (K)
- net at U4.8 (LED2): now also R48.2; no longer D48.1 (K)
- net at U4.9 (LED3): now also R49.2; no longer D49.1 (K)
- net SWCLC renamed SWCLK
- net SWCLK: now also J2.4 (SWCLK)
- new net: D1.1 (K), R1.1
- new net: D2.1 (K), R2.1
- new net: D3.1 (K), R3.1
- new net: D4.1 (K), R4.1
- new net: D5.1 (K), R5.1
- new net: D6.1 (K), R6.1
- new net: D7.1 (K), R7.1
- new net: D8.1 (K), R8.1
- new net: D9.1 (K), R9.1
- new net: D10.1 (K), R10.1
- new net: D11.1 (K), R11.1
- new net: D12.1 (K), R12.1
- new net: D13.1 (K), R13.1
- new net: D14.1 (K), R14.1
- new net: D15.1 (K), R15.1
- new net: D16.1 (K), R16.1
- new net: D17.1 (K), R17.1
- new net: D18.1 (K), R18.1
- new net: D19.1 (K), R19.1
- new net: D20.1 (K), R20.1
- new net: D21.1 (K), R21.1
- new net: D22.1 (K), R22.1
- new net: D23.1 (K), R23.1
- new net: D24.1 (K), R24.1
- new net: D25.1 (K), R25.1
- new net: D26.1 (K), R26.1
- new net: D27.1 (K), R27.1
- new net: D28.1 (K), R28.1
- new net: D29.1 (K), R29.1
- new net: D30.1 (K), R30.1
- new net: D31.1 (K), R31.1
- new net: D32.1 (K), R32.1
- new net: D33.1 (K), R33.1
- new net: D34.1 (K), R34.1
- new net: D35.1 (K), R35.1
- new net: D36.1 (K), R36.1
- new net: D37.1 (K), R37.1
- new net: D38.1 (K), R38.1
- new net: D39.1 (K), R39.1
- new net: D40.1 (K), R40.1
- new net: D41.1 (K), R41.1
- new net: D42.1 (K), R42.1
- new net: D43.1 (K), R43.1
- new net: D44.1 (K), R44.1
- new net: D45.1 (K), R45.1
- new net: D46.1 (K), R46.1
- new net: D47.1 (K), R47.1
- new net: D48.1 (K), R48.1
- new net: D49.1 (K), R49.1
- new net: D50.1 (K), R50.1
- new net: D51.1 (K), R51.1
- new net: D52.1 (K), R52.1
- new net: D53.1 (K), R53.1
- new net: D54.1 (K), R54.1
- new net: D55.1 (K), R55.1
- new net: D56.1 (K), R56.1
- new net: D57.1 (K), R57.1
- new net: D58.1 (K), R58.1
- new net: D59.1 (K), R59.1
- new net: D60.1 (K), R60.1
- no-connect marks 15 -> 13
Other:
- moved on the sheet: D1, D10, D11, D12, D13, D14, D15, D16, D17, D18, D19, D2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
